File: monaco-gp.kicad_sch (KiCad schematic)
At the start: 4 parts

Commit message: correct footprints in schematic
Parts:
- B1: footprint Library:Edge2x22_3.95mm -> Library:Edge2x22_3.95mm_top
- E1: footprint Library:Edge2x22_3.95mm -> Library:Edge2x22_3.95mm_bottom
Changed lines of the file:
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@@
 			)
 		)
-		(property "Footprint" "Library:Edge2x22_3.95mm"
+		(property "Footprint" "Library:Edge2x22_3.95mm_bottom"
 			(at 160.02 44.45 0)
 			(effects
@@
 			)
 		)
-		(property "Footprint" "Library:Edge2x22_3.95mm"
+		(property "Footprint" "Library:Edge2x22_3.95mm_top"
 			(at 160.02 78.74 0)
 			(effects

Commit message: .
Parts:
- B1: footprint Library:Edge2x22_3.95mm_top -> Library:Edge2x22_3.95mm_bottom
- E1: footprint Library:Edge2x22_3.95mm_bottom -> Library:Edge2x22_3.95mm_top
Changed lines of the file:
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@@
 			)
 		)
-		(property "Footprint" "Library:Edge2x22_3.95mm_bottom"
+		(property "Footprint" "Library:Edge2x22_3.95mm_top"
 			(at 160.02 44.45 0)
 			(effects
@@
 			)
 		)
-		(property "Footprint" "Library:Edge2x22_3.95mm_top"
+		(property "Footprint" "Library:Edge2x22_3.95mm_bottom"
 			(at 160.02 78.74 0)
 			(effects

Commit message: .
Parts:
- B1: footprint Library:Edge2x22_3.95mm_bottom -> Library:Edge2x22_3.95mm_top
- E1: footprint Library:Edge2x22_3.95mm_top -> Library:Edge2x22_3.95mm_bottom
Changed lines of the file:
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@@
 			)
 		)
-		(property "Footprint" "Library:Edge2x22_3.95mm_top"
+		(property "Footprint" "Library:Edge2x22_3.95mm_bottom"
 			(at 160.02 44.45 0)
 			(effects
@@
 			)
 		)
-		(property "Footprint" "Library:Edge2x22_3.95mm_bottom"
+		(property "Footprint" "Library:Edge2x22_3.95mm_top"
 			(at 160.02 78.74 0)
 			(effects
